File: arcticfoxlight.kicad_sch (KiCad schematic)
At the start: 9 parts, among them J1 USB_C_Receptacle_USB2.0_16P, SW1 SW_Push, U2 ESP32-C6-MINI-1/U, U3 LM2596S-3.3

Commit message: Day 2
Parts:
- removed C4: 0.1uF, Capacitor_SMD:C_0402_1005Metric, symbol Device:C
- removed SW1: SW_Push, symbol Switch:SW_Push
- added C1, C13: 10uF, Capacitor_SMD:C_0805_2012Metric_Pad1.18x1.45mm_HandSolder, symbol Device:C
- added C12, C14: 100nF, Capacitor_SMD:C_0805_2012Metric_Pad1.18x1.45mm_HandSolder, symbol Device:C
- added R10, R8, R9: R10k, Resistor_SMD:R_0201_0603Metric_Pad0.64x0.40mm_HandSolder, symbol Device:R
- added R4, R5: 10k, Resistor_SMD:R_0805_2012Metric_Pad1.20x1.40mm_HandSolder, symbol Device:R_US
- added R6: R27O, Resistor_SMD:R_0201_0603Metric_Pad0.64x0.40mm_HandSolder, symbol Device:R
- added R7: R330o, Resistor_SMD:R_0201_0603Metric_Pad0.64x0.40mm_HandSolder, symbol Device:R
- added SW1: RESET, Button_Switch_SMD:SW_SPST_TL3342, symbol C5117870_lib:GT-TC060A-H025-L1
- added SW2: FLASH, Button_Switch_SMD:SW_SPST_TL3342, symbol C5117870_lib:GT-TC060A-H025-L1
- added U1: LM2596S-5, Package_TO_SOT_SMD:TO-263-5_TabPin3, symbol Regulator_Switching:LM2596S-5
- added U4: SN74AHCT125N, footprints:DIP794W45P254L1930H508Q14, symbol SN74AHCT125N:SN74AHCT125N
- J1: footprint (none) -> Connector_USB:USB_C_Receptacle_HCTL_HC-TYPE-C-16P-01A
- R1, R2: footprint (none) -> Resistor_SMD:R_0201_0603Metric_Pad0.64x0.40mm_HandSolder
- R3: value R10K -> R27O; footprint (none) -> Resistor_SMD:R_0201_0603Metric_Pad0.64x0.40mm_HandSolder
- U2: footprint PCM_Espressif:ESP32-C6-MINI-1 -> Espressif:ESP32-C6-MINI-1
Connections:
- net D+: now also R6.2; no longer J1.A6 (D+), J1.B6 (D+)
- net D-: now also R3.2; no longer J1.A7 (D-), J1.B7 (D-)
- net GND: now also D1.3 (VSS), U2.1 (GND), U2.11 (GND), U2.14 (GND), U2.2 (GND), U2.36 (GND), U2.37 (GND), U2.38 (GND), U2.39 (GND), U2.40 (GND), U2.41 (GND), U2.42 (GND), U2.43 (GND), U2.44 (GND), U2.45 (GND), U2.46 (GND), U2.47 (GND), U2.48 (GND), U2.49 (GND), U2.50 (GND), U2.51 (GND), U2.52 (GND), U2.53 (GND), U3.3 (GND), U3.5 (~{ON}/OFF), C1.2, C12.2, C13.2, C14.2, R10.1, R8.1, R9.1, SW1.1, SW2.1, U1.3 (GND), U1.5 (~{ON}/OFF), U4.1 (1~{OE}), U4.7 (GND)
- net VCC: now also U3.1 (VIN), U1.1 (VIN)
- net +3.3V: now reaches U3.2 (OUT)
- net +3.3V: now also U2.3 (3V3), U3.4 (FB), C1.1, C12.1, C13.1, R4.2, R5.1
- net +5V: now reaches D1.1 (VDD)
- net +5V: now also U1.2 (OUT), U1.4 (FB), U4.10 (3~{OE}), U4.13 (4~{OE}), U4.14 (VCC), U4.4 (2~{OE})
- net at D1.4 (DIN): now also U4.3 (1Y)
- net at U2.10 (MTDI/GPIO5/ADC1_CH5): now also R7.2
- net BOOT: now reaches U2.12 (GPIO0/ADC1_CH0/XTAL_32K_P)
- net BOOT: now also R4.1, SW2.2
- net +3V3: no longer names the net of R3.1
- net +3V3: now also J1.A7 (D-), J1.B7 (D-); no longer U2.3 (3V3)
- net ENABLE renamed EN
- net EN: now also C14.1, R5.2, SW1.2; no longer R3.2
- new net: R10.2, U4.12 (4A)
- new net: R8.2, U4.5 (2A)
- new net: R9.2, U4.9 (3A)
- new net: J1.A6 (D+), J1.B6 (D+), R6.1
- new net DIN: R7.1, U4.2 (1A)
- no-connect marks 6 -> 24
Other:
- note added: "LED"
- note added: "LED Power"
- note added: "MCU"
- note added: "MCU Power"
- note added: "USB C"
- moved on the sheet: D1, U2, U3

Commit message: Day 2.1
Parts:
- removed C14: 100nF, Capacitor_SMD:C_0805_2012Metric_Pad1.18x1.45mm_HandSolder, symbol Device:C
- removed R4, R5: 10k, Resistor_SMD:R_0805_2012Metric_Pad1.20x1.40mm_HandSolder, symbol Device:R_US
- removed SW1: RESET, Button_Switch_SMD:SW_SPST_TL3342, symbol C5117870_lib:GT-TC060A-H025-L1
- removed SW2: FLASH, Button_Switch_SMD:SW_SPST_TL3342, symbol C5117870_lib:GT-TC060A-H025-L1
- added H1: MountingHole, MountingHole:MountingHole_2.2mm_M2, symbol Mechanical:MountingHole
Connections:
- net BOOT: no longer names the net of U2.12 (GPIO0/ADC1_CH0/XTAL_32K_P)
- net EN: no longer names the net of U2.8 (EN/CHIP_PU)
- no-connect marks 24 -> 26
